Commit message: URDF modificado do Caio e lógica de desvio aprimorada

File: description/robot.urdf.xacro (robot description, xacro)
@@ -66,6 +66,6 @@
   </link>
   <joint name="base_joint" type="fixed">
-    <parent link="base_link"/>
-    <child link="base_footprint"/>
+    <parent link="base_footprint"/>
+    <child link="base_link"/>
     <origin xyz="0.0 0.0 ${-(wheel_radius+wheel_zoff)}" rpy="0 0 0"/>
   </joint>
@@ -246,8 +246,10 @@
     <joint name="gripper_extension">
       <command_interface name="position">
-        <param name="min">-1.57075</param>
-        <param name="max">0.2</param>
+        <param name="min">0.0</param>
+        <param name="max">0.4</param>
       </command_interface>
-      <state_interface name="position"/>
+      <state_interface name="position">
+        <param name="initial_value">0.0</param>
+      </state_interface>
       <state_interface name="velocity"/>
     </joint>
@@ -257,5 +259,7 @@
         <param name="max">0.06</param>
       </command_interface>
-      <state_interface name="position"/>
+      <state_interface name="position">
+        <param name="initial_value">0.0</param>
+      </state_interface>
       <state_interface name="velocity"/>
     </joint>
@@ -265,5 +269,7 @@
         <param name="max">0.0</param>
       </command_interface>
-      <state_interface name="position"/>
+      <state_interface name="position">
+        <param name="initial_value">0.0</param>
+      </state_interface>
       <state_interface name="velocity"/>
     </joint>
@@ -469,7 +475,7 @@
     </sensor> -->
   </gazebo>
-  <joint name="gripper_extension" type="revolute">
-    <axis xyz="0 1 0"/>
-    <limit effort="50.0" lower="-1.57075" upper="0.2" velocity="0.5"/>
+  <joint name="gripper_extension" type="prismatic">
+    <axis xyz="1 0 0"/>
+    <limit effort="50.0" lower="0.0" upper="0.4" velocity="0.5"/>
     <origin rpy="0 0 0" xyz="0.2 0 0.1"/>
     <parent link="base_link"/>
@@ -479,11 +485,12 @@
     <visual>
       <geometry>
-        <cylinder length="0.2" radius="0.01"/>
-      </geometry>
-      <origin rpy="0 1.57075 0" xyz="0.1 0 0"/>
-    </visual>
-    <collision>
-      <geometry>
-        <cylinder length="0.2" radius="0.01"/>
+        <cylinder length="0.4" radius="0.01"/>
+      </geometry>
+      <origin rpy="0 1.57075 0" xyz="-0.18 0 -0.1"/>
+    </visual>
+    <collision>
+      <origin rpy="0 1.57075 0" xyz="-0.18 0 -0.1"/>
+      <geometry>
+        <cylinder length="0.4" radius="0.01"/>
       </geometry>
     </collision>
@@ -499,4 +506,5 @@
   <link name="left_gripper">
     <visual>
+      <origin rpy="-3.1415 0 0" xyz="-0.13 0 -0.1"/>
       <geometry>
         <box size="0.1 0.02 0.02"/> <!-- Comprimento, largura, altura -->
@@ -504,4 +512,5 @@
     </visual>
     <collision>
+      <origin rpy="-3.1415 0 0" xyz="-0.13 0 -0.1"/>
       <geometry>
         <box size="0.1 0.02 0.02"/>
@@ -517,5 +526,5 @@
   <link name="left_tip">
     <visual>
-      <origin rpy="0 0 -0.1" xyz="0.03 0 0"/>
+      <origin rpy="0 0 -0.1" xyz="-0.1 0 -0.1"/>
       <geometry>
         <box size="0.06 0.01 0.01"/>
@@ -523,5 +532,5 @@
     </visual>
     <collision>
-      <origin rpy="0 0 -0.1" xyz="0.03 0 0"/>
+      <origin rpy="0 0 -0.1" xyz="-0.1 0 -0.1"/>
       <geometry>
         <box size="0.06 0.01 0.01"/>
@@ -539,5 +548,5 @@
   <link name="right_gripper">
     <visual>
-      <origin rpy="-3.1415 0 0" xyz="0 0 0"/>
+      <origin rpy="-3.1415 0 0" xyz="-0.13 0 -0.1"/>
       <geometry>
         <box size="0.1 0.02 0.02"/>
@@ -545,5 +554,5 @@
     </visual>
     <collision>
-      <origin rpy="-3.1415 0 0" xyz="0 0 0"/>
+      <origin rpy="-3.1415 0 0" xyz="-0.13 0 -0.1"/>
       <geometry>
         <box size="0.1 0.02 0.02"/>
@@ -553,5 +562,5 @@
   </link>
   <joint name="right_tip_joint" type="fixed">
-    <origin rpy="-3.1415 0 0" xyz="0.06 -0.001 0"/>
+    <origin rpy="0.0 0 0" xyz="0.06 -0.001 0"/>
     <parent link="right_gripper"/>
     <child link="right_tip"/>
@@ -559,5 +568,5 @@
   <link name="right_tip">
     <visual>
-      <origin rpy="0 0 -0.1" xyz="0.03 0 0"/>
+      <origin rpy="0 0 0.1" xyz="-0.1 0 -0.1"/>
       <geometry>
         <box size="0.06 0.01 0.01"/>
@@ -565,5 +574,5 @@
     </visual>
     <collision>
-      <origin rpy="0 0 -0.1" xyz="0.03 0 0"/>
+      <origin rpy="0 0 0.1" xyz="-0.1 0 -0.1"/>
       <geometry>
         <box size="0.06 0.01 0.01"/>

Commit message: PERRY

File: description/robot.urdf.xacro (robot description, xacro)
@@ -256,6 +256,6 @@
     <joint name="left_gripper_joint">
       <command_interface name="position">
-        <param name="min">0.0</param>
-        <param name="max">0.06</param>
+        <param name="min">-1.57</param>
+        <param name="max">1.57</param>
       </command_interface>
       <state_interface name="position">
@@ -266,6 +266,26 @@
     <joint name="right_gripper_joint">
       <command_interface name="position">
-        <param name="min">-0.06</param>
-        <param name="max">0.0</param>
+        <param name="min">-1.57</param>
+        <param name="max">1.57</param>
+      </command_interface>
+      <state_interface name="position">
+        <param name="initial_value">0.0</param>
+      </state_interface>
+      <state_interface name="velocity"/>
+    </joint>
+    <joint name="left_tip_joint">
+      <command_interface name="position">
+        <param name="min">-1.57</param>
+        <param name="max">1.57</param>
+      </command_interface>
+      <state_interface name="position">
+        <param name="initial_value">0.0</param>
+      </state_interface>
+      <state_interface name="velocity"/>
+    </joint>
+    <joint name="right_tip_joint">
+      <command_interface name="position">
+        <param name="min">-1.57</param>
+        <param name="max">1.57</param>
       </command_interface>
       <state_interface name="position">
@@ -297,6 +317,6 @@
         <cylinder radius="0.0508" length="0.055"/>
       </geometry>
-      <material name="LightBlue">
-        <color rgba="0.11 0.37 0.56 1.0"/>
+      <material name="DarkBrown">
+        <color rgba="0.25 0.08 0.03 1.0"/>
       </material>
     </visual>
@@ -477,6 +497,7 @@
   <joint name="gripper_extension" type="prismatic">
     <axis xyz="1 0 0"/>
-    <limit effort="50.0" lower="0.0" upper="0.4" velocity="0.5"/>
+    <limit effort="100.0" lower="0.0" upper="0.4" velocity="0.5"/>
     <origin rpy="0 0 0" xyz="0.2 0 0.1"/>
+    <dynamics damping="1.0" friction="0.5"/>
     <parent link="base_link"/>
     <child link="gripper_pole"/>
@@ -488,4 +509,7 @@
       </geometry>
       <origin rpy="0 1.57075 0" xyz="-0.18 0 -0.1"/>
+      <material name="orange">
+        <color rgba="1.0 0.4 0 1.0"/>
+      </material>
     </visual>
     <collision>
@@ -497,20 +521,24 @@
     <xacro:cylinder_inertia m="0.01" r="0.01" h="0.2"/>
   </link>
-  <joint name="left_gripper_joint" type="prismatic">
-    <axis xyz="0 1 0"/>
-    <limit effort="100.0" lower="0.0" upper="0.06" velocity="0.25"/>
-    <origin rpy="0 0 0" xyz="0.2 0.01 0"/>
-    <parent link="gripper_pole"/>
+  <joint name="left_gripper_joint" type="revolute">
+   <axis xyz="0 0 1"/>
+    <limit effort="500.0" lower="-1.57" upper="1.57" velocity="0.25"/>
+    <origin rpy="0 0 0" xyz="0.025 0.015 -0.1"/>
+    <dynamics damping="1.0" friction="0.5"/>
+    <parent link="gear"/>
     <child link="left_gripper"/>
   </joint>
   <link name="left_gripper">
     <visual>
-      <origin rpy="-3.1415 0 0" xyz="-0.13 0 -0.1"/>
+      <origin rpy="0 0 0" xyz="0.05 0.0 0.0"/>
       <geometry>
         <box size="0.1 0.02 0.02"/> <!-- Comprimento, largura, altura -->
       </geometry>
-    </visual>
-    <collision>
-      <origin rpy="-3.1415 0 0" xyz="-0.13 0 -0.1"/>
+      <material name="orange">
+        <color rgba="1.0 0.4 0 1.0"/>
+      </material>
+    </visual>
+    <collision>
+      <origin rpy="0 0 0" xyz="0.05 0.0 0.0"/>
       <geometry>
         <box size="0.1 0.02 0.02"/>
@@ -519,6 +547,9 @@
     <xacro:box_inertia m="0.015" w="0.02" h="0.02" d="0.1"/>
   </link>
-  <joint name="left_tip_joint" type="fixed">
-    <origin rpy="0.0 0 0" xyz="0.06 0.001 0"/>
+  <joint name="left_tip_joint" type="revolute">
+    <origin rpy="0 0 0" xyz="0.1 0.001 0"/>
+    <axis xyz="0 0 1"/>
+    <limit effort="100.0" lower="-1.57" upper="1.57" velocity="0.25"/>
+    <dynamics damping="1.0" friction="0.5"/>
     <parent link="left_gripper"/>
     <child link="left_tip"/>
@@ -526,11 +557,14 @@
   <link name="left_tip">
     <visual>
-      <origin rpy="0 0 -0.1" xyz="-0.1 0 -0.1"/>
+      <origin rpy="0 0 -0.1" xyz="0.03 0 0"/>
       <geometry>
         <box size="0.06 0.01 0.01"/>
       </geometry>
-    </visual>
-    <collision>
-      <origin rpy="0 0 -0.1" xyz="-0.1 0 -0.1"/>
+      <material name="orange">
+        <color rgba="1.0 0.4 0 1.0"/>
+      </material>
+    </visual>
+    <collision>
+      <origin rpy="0 0 0" xyz="0.03 0 0"/>
       <geometry>
         <box size="0.06 0.01 0.01"/>
@@ -539,20 +573,24 @@
     <xacro:box_inertia m="0.005" w="0.01" h="0.01" d="0.06"/>
   </link>
-  <joint name="right_gripper_joint" type="prismatic">
-    <axis xyz="0 1 0"/>
-    <limit effort="100.0" lower="-0.06" upper="0" velocity="0.25"/>
-    <origin rpy="0 0 0" xyz="0.2 -0.01 0"/>
-    <parent link="gripper_pole"/>
+  <joint name="right_gripper_joint" type="revolute">
+    <axis xyz="0 0 -1"/>
+    <limit effort="500.0" lower="-1.57" upper="1.57" velocity="0.25"/>
+    <origin rpy="0 0 0" xyz="0.025 -0.015 -0.1"/>
+    <dynamics damping="1.0" friction="0.5"/>
+    <parent link="gear"/>
     <child link="right_gripper"/>
   </joint>
   <link name="right_gripper">
     <visual>
-      <origin rpy="-3.1415 0 0" xyz="-0.13 0 -0.1"/>
+      <origin rpy="0 0 0" xyz="0.05 0.0 0.0"/>
       <geometry>
         <box size="0.1 0.02 0.02"/>
       </geometry>
-    </visual>
-    <collision>
-      <origin rpy="-3.1415 0 0" xyz="-0.13 0 -0.1"/>
+      <material name="orange">
+        <color rgba="1.0 0.4 0 1.0"/>
+      </material>
+    </visual>
+    <collision>
+      <origin rpy="0 0 0" xyz="0.05 0.0 0.0"/>
       <geometry>
         <box size="0.1 0.02 0.02"/>
@@ -561,6 +599,9 @@
     <xacro:box_inertia m="0.015" w="0.02" h="0.02" d="0.1"/>
   </link>
-  <joint name="right_tip_joint" type="fixed">
-    <origin rpy="0.0 0 0" xyz="0.06 -0.001 0"/>
+  <joint name="right_tip_joint" type="revolute">
+    <origin rpy="0 0 0" xyz="0.1 -0.001 0"/>
+    <axis xyz="0 0 -1"/>
+    <limit effort="100.0" lower="-1.57" upper="1.57" velocity="0.25"/>
+    <dynamics damping="1.0" friction="0.5"/>
     <parent link="right_gripper"/>
     <child link="right_tip"/>
@@ -568,11 +609,14 @@
   <link name="right_tip">
     <visual>
-      <origin rpy="0 0 0.1" xyz="-0.1 0 -0.1"/>
+      <origin rpy="0 0 0.1" xyz="0.03 0 0"/>
       <geometry>
         <box size="0.06 0.01 0.01"/>
       </geometry>
-    </visual>
-    <collision>
-      <origin rpy="0 0 0.1" xyz="-0.1 0 -0.1"/>
+      <material name="orange">
+        <color rgba="1.0 0.4 0 1.0"/>
+      </material>
+    </visual>
+    <collision>
+      <origin rpy="0 0 0" xyz="0.03 0 0"/>
       <geometry>
         <box size="0.06 0.01 0.01"/>
@@ -581,3 +625,103 @@
     <xacro:box_inertia m="0.005" w="0.01" h="0.01" d="0.06"/>
   </link>
+  <!-- <link name="left_gear">
+    <visual>
+      <origin rpy="0 0 0" xyz= "0.025 0.012 -0.1"/>
+        <geometry>
+          <sphere radius="0.01"/>
+        </geometry>
+        <material name="orange">
+        <color rgba="1.0 0.4 0 1.0"/>
+      </material>
+    </visual>
+    <xacro:sphere_inertia m="0.005" r="0.1"/>
+  </link>
+  <joint name="left_gear_joint" type="fixed">
+    <origin rpy="0 0 0" xyz="0 0 0"/>
+    <parent link="gripper_pole"/>
+    <child link="left_gear"/>
+  </joint>
+    <link name="right_gear">
+    <visual>
+      <origin rpy="0 0 0" xyz= "0.025 -0.012 -0.1"/>
+        <geometry>
+          <sphere radius="0.01"/>
+        </geometry>
+        <material name="orange">
+        <color rgba="1.0 0.4 0 1.0"/>
+      </material>
+    </visual>
+    <xacro:sphere_inertia m="0.005" r="0.1"/>
+  </link>
+  <joint name="right_gear_joint" type="fixed">
+    <origin rpy="0 0 0" xyz="0 0 0"/>
+    <parent link="gripper_pole"/>
+    <child link="right_gear"/>
+  </joint> -->
+  <link name="gear">
+    <visual>
+      <origin rpy="0 0 0" xyz= "0.025 0.0 -0.1"/>
+        <geometry>
+          <sphere radius="0.015"/>
+        </geometry>
+        <material name="orange">
+        <color rgba="1.0 0.4 0 1.0"/>
+      </material>
+    </visual>
+    <xacro:sphere_inertia m="0.005" r="0.1"/>
+  </link>
+  <joint name="gear_joint" type="fixed">
+    <origin rpy="0 0 0" xyz="0 0 0"/>
+    <parent link="gripper_pole"/>
+    <child link="gear"/>
+  </joint>
+    <link name="tale">
+    <visual>
+      <geometry>
+        <box size="${base_length/2} ${base_width*0.7} ${base_height/5}"/>
+      </geometry>
+      <material name="brown">
+        <color rgba="1.0 0.5 0 1.0"/>
+      </material>
+    </visual>
+    <collision>
+      <geometry>
+        <box size="${base_length/2} ${base_width*0.7} ${base_height/5}"/>
+      </geometry>
+    </collision>
+    <xacro:box_inertia m="0.001" w="${base_length/2}" d="${base_width*0.7}" h="${base_height/5}"/>
+  </link>
+  <joint name="tale_joint" type="fixed">
+    <parent link="base_footprint"/>
+    <child link="tale"/>
+    <origin xyz="-${base_length*0.7} 0.0 -${base_height}" rpy="0 0 0"/>
+  </joint>
+    <link name="left_eye">
+    <visual>
+      <origin rpy="0 0 0" xyz= "0.21 0.1 -0.1"/>
+        <geometry>
+          <sphere radius="0.01"/>
+        </geometry>
+    </visual>
+    <xacro:sphere_inertia m="0.005" r="0.1"/>
+  </link>
+  <joint name="left_eye_joint" type="fixed">
+    <origin rpy="0 0 0" xyz="0 0 0"/>
+    <parent link="base_footprint"/>
+    <child link="left_eye"/>
+  </joint>
+    <link name="right_eye">
+    <visual>
+      <origin rpy="0 0 0" xyz= "0.21 -0.1 -0.1"/>
+        <geometry>
+          <sphere radius="0.01"/>
+        </geometry>
+    </visual>
+    <xacro:sphere_inertia m="0.005" r="0.1"/>
+  </link>
+  <joint name="right_eye_joint" type="fixed">
+    <origin rpy="0 0 0" xyz="0 0 0"/>
+    <parent link="base_footprint"/>
+    <child link="right_eye"/>
+  </joint>
 </robot>

Commit message: PERRY COM OLHOS

File: description/robot.urdf.xacro (robot description, xacro)
@@ -701,8 +701,11 @@
       <origin rpy="0 0 0" xyz= "0.21 0.1 -0.1"/>
         <geometry>
-          <sphere radius="0.01"/>
-        </geometry>
-    </visual>
-    <xacro:sphere_inertia m="0.005" r="0.1"/>
+          <sphere radius="0.018"/>
+        </geometry>
+        <material name="white">
+        <color rgba="1.0 1.0 1.0 1.0"/>
+      </material>
+    </visual>
+    <xacro:sphere_inertia m="0.005" r="0.13"/>
   </link>
   <joint name="left_eye_joint" type="fixed">
@@ -715,8 +718,11 @@
       <origin rpy="0 0 0" xyz= "0.21 -0.1 -0.1"/>
         <geometry>
-          <sphere radius="0.01"/>
-        </geometry>
-    </visual>
-    <xacro:sphere_inertia m="0.005" r="0.1"/>
+          <sphere radius="0.018"/>
+        </geometry>
+        <material name="white">
+        <color rgba="1.0 1.0 1.0 1.0"/>
+      </material>
+    </visual>
+    <xacro:sphere_inertia m="0.005" r="0.13"/>
   </link>
   <joint name="right_eye_joint" type="fixed">
@@ -725,3 +731,31 @@
     <child link="right_eye"/>
   </joint>
+  <link name="left_eye_two">
+    <visual>
+      <origin rpy="0 0 0" xyz= "0.215 0.105 -0.1"/>
+        <geometry>
+          <sphere radius="0.014"/>
+        </geometry>
+    </visual>
+    <xacro:sphere_inertia m="0.005" r="0.006"/>
+  </link>
+  <joint name="left_eye_two_joint" type="fixed">
+    <origin rpy="0 0 0" xyz="0 0 0"/>
+    <parent link="base_footprint"/>
+    <child link="left_eye_two"/>
+  </joint>
+    <link name="right_eye_two">
+    <visual>
+      <origin rpy="0 0 0" xyz= "0.215 -0.105 -0.1"/>
+        <geometry>
+          <sphere radius="0.014"/>
+        </geometry>
+    </visual>
+    <xacro:sphere_inertia m="0.005" r="0.006"/>
+  </link>
+  <joint name="right_eye_two_joint" type="fixed">
+    <origin rpy="0 0 0" xyz="0 0 0"/>
+    <parent link="base_footprint"/>
+    <child link="right_eye_two"/>
+  </joint>
 </robot>
